File: xover-psu.kicad_pcb (KiCad board)
At the start: 2 copper layers, 100 x 100 mm, 113 parts, among them J1 Screw_Terminal_01x02, J2 Screw_Terminal_01x02, J3 Screw_Terminal_01x02, J4 Screw_Terminal_01x03, J5 Screw_Terminal_01x03, J6 Screw_Terminal_01x03, J7 Screw_Terminal_01x03, J8 Screw_Terminal_01x02, J9 Screw_Terminal_01x02, K1 T9GS1L14-12, Q1 AO3400, Q2 2N7002, Q3 AO3401A, U1 817C, U2 817C, U3 TL431DBZ, U4 LM317_3PinPackage, U5 LM337_TO220, U6 817C, U7 TL431DBZ

Commit message: tested UNMUTE circuit, improved switch-on/off speed, rejigged mains routing for EMI
Parts:
- added REF**: Symbol_Highvoltage_Type2_FSilk_Small, pcb:Symbol_Highvoltage_Type2_FSilk_Small, F.Cu at (40.8, 75.0)
- added REF**: Tyrrell Zaibatsu, tz:Tyrrell-Zaibatsu-20-Back, F.Cu at (107.5, 101.5)
- added REF**: Tyrrell Zaibatsu, tz:Tyrrell-Zaibatsu-10, F.Cu at (86.5, 74.0)
- added REF***: OSHW-Symbol_6.7x6mm_SilkScreen, pcb:OSHW-Symbol_6.7x6mm_BackSilkScreen, F.Cu at (89.2, 71.5)
- K1: value T9GS1L14-12 -> T9GS1L24-12
- R18, R28: value 240 -> 270
- R20, R23: value 4k3 -> 5k1
- R21, R24: value 4k3 -> 6k8
- R35: value 680 -> 1k
- U1, U2, U6: footprint Housings_DIP:DIP-4_W7.62mm_Socket -> Housings_DIP:DIP-4_W7.62mm
- moved R3 84.6 mm to (92.8, 52.2), turned to 90 degrees
- moved R2 77.2 mm to (85.2, 43.8), turned to 90 degrees
- moved U3 76.2 mm to (99.5, 56.0), turned to 90 degrees
- moved R7 75.6 mm to (94.8, 52.2), turned to 90 degrees
- moved R11 73.8 mm to (106.5, 54.8)
- moved R12 72.6 mm to (100.0, 52.2), turned to 90 degrees
- moved Q2 72.3 mm to (95.5, 56.0), turned to 90 degrees
- moved R36 69.4 mm to (103.0, 54.8)
- moved C2 68.0 mm to (106.0, 57.5)
- moved R1 66.2 mm to (99.5, 60.2)
- moved R13 65.8 mm to (90.8, 52.2), turned to 270 degrees
- moved R35 64.2 mm to (91.8, 60.2), turned to 0 degrees
- moved R5 64.1 mm to (102.5, 57.5), turned to 90 degrees
- moved U7 63.6 mm to (91.5, 56.0), turned to 90 degrees
- moved R34 62.8 mm to (88.8, 52.2), turned to 90 degrees
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Routing:
- net Net-(D2-Pad2): track 0.00 -> 69.7 mm, vias 0 -> 2
- net /NEUTRAL: track 112.9 -> 179.3 mm, vias 0 -> 3
- net Net-(D5-Pad2): track 0.00 -> 44.1 mm
- net /VDD: track 124.4 -> 159.8 mm
- net Net-(C1-Pad1): track 0.00 -> 20.0 mm
- net Net-(Q2-Pad1): track 0.00 -> 10.5 mm
- net Net-(Q3-Pad1): track 0.00 -> 9.59 mm
- net Net-(R1-Pad1): track 0.00 -> 7.33 mm
- net Net-(C2-Pad1): track 0.00 -> 7.18 mm
- net /PRI: track 54.8 -> 61.6 mm
- net Net-(R34-Pad1): track 0.00 -> 6.35 mm
- net Net-(R35-Pad2): track 0.00 -> 4.14 mm
- net Net-(R13-Pad1): track 0.00 -> 4.00 mm
- net Net-(D6-Pad1): track 0.00 -> 3.70 mm
- net Net-(R36-Pad1): track 0.00 -> 3.26 mm
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Other:
- outline, holes or cut-outs redrawn
- net class AC: clearance 2 -> 1.95
- board text added: "+"
- board text removed: "DC12"

Commit message: taped out, updated README
Parts:
- added FID1: Fiducial, Fiducials:Fiducial_1mm_Dia_2.54mm_Outer_CopperTop, F.Cu at (109.0, 33.5)
- added FID2: Fiducial, Fiducials:Fiducial_1mm_Dia_2.54mm_Outer_CopperTop, F.Cu at (33.0, 115.0)
- added FID3: Fiducial, Fiducials:Fiducial_1mm_Dia_2.54mm_Outer_CopperTop, F.Cu at (99.0, 120.0)
- added FID4: Fiducial, Fiducials:Fiducial_1mm_Dia_2.54mm_Outer_CopperTop, F.Cu at (54.0, 30.0)
Routing:
- net /RECT2B: track 91.0 -> 85.0 mm
- net /RECT2: track 37.1 -> 31.1 mm
- net /RECT1: track 64.7 -> 58.7 mm
- net /RECT1B: track 99.4 -> 93.4 mm
