File: xover-psu.sch (KiCad schematic (older format))
At the start: 113 parts, among them J1 Screw_Terminal_01x02, J2 Screw_Terminal_01x02, J3 Screw_Terminal_01x02, J4 Screw_Terminal_01x03, J5 Screw_Terminal_01x03, J6 Screw_Terminal_01x03, J7 Screw_Terminal_01x03, J8 Screw_Terminal_01x02, J9 Screw_Terminal_01x02, K1 T9GS1L24-12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

Commit message: taped out, updated README
Parts:
- added FID1, FID2, FID3, FID4: Fiducial, Fiducials:Fiducial_1mm_Dia_2.54mm_Outer_CopperTop, symbol Mechanical:Fiducial
Changed lines of the file:
@@
 Wire Wire Line
 	4200 5150 5050 5150
+$Comp
+L Mechanical:Fiducial FID1
+U 1 1 617B9046
+P 900 700
+F 0 "FID1" H 985 746 50  0000 L CNN
+F 1 "Fiducial" H 985 655 50  0000 L CNN
+F 2 "Fiducials:Fiducial_1mm_Dia_2.54mm_Outer_CopperTop" H 900 700 50  0001 C CNN
+F 3 "~" H 900 700 50  0001 C CNN
+	1    900  700
+	1    0    0    -1
+$EndComp
+$Comp
+L Mechanical:Fiducial FID3
+U 1 1 617F39FF
+P 900 900
+F 0 "FID3" H 985 946 50  0000 L CNN
+F 1 "Fiducial" H 985 855 50  0000 L CNN
+F 2 "Fiducials:Fiducial_1mm_Dia_2.54mm_Outer_CopperTop" H 900 900 50  0001 C CNN
+F 3 "~" H 900 900 50  0001 C CNN
+	1    900  900
+	1    0    0    -1
+$EndComp
+$Comp
+L Mechanical:Fiducial FID2
+U 1 1 617F4321
+P 1150 700
+F 0 "FID2" H 1235 746 50  0000 L CNN
+F 1 "Fiducial" H 1235 655 50  0000 L CNN
+F 2 "Fiducials:Fiducial_1mm_Dia_2.54mm_Outer_CopperTop" H 1150 700 50  0001 C CNN
+F 3 "~" H 1150 700 50  0001 C CNN
+	1    1150 700
+	1    0    0    -1
+$EndComp
+$Comp
+L Mechanical:Fiducial FID4
+U 1 1 617F4BE5
+P 1150 900
+F 0 "FID4" H 1235 946 50  0000 L CNN
+F 1 "Fiducial" H 1235 855 50  0000 L CNN
+F 2 "Fiducials:Fiducial_1mm_Dia_2.54mm_Outer_CopperTop" H 1150 900 50  0001 C CNN
+F 3 "~" H 1150 900 50  0001 C CNN
+	1    1150 900
+	1    0    0    -1
+$EndComp
 $EndSCHEMATC
